Commit message: Adapt COLT URDF and Xacro to legged_control interfaces

File: src/colt/urdf/colt.urdf (robot description, URDF)
Before this commit: robot colt, 18 links, 17 joints
Links:
- removed link C_LF_FOOT
- removed link C_LF_HAA
- removed link C_LF_HFE
- removed link C_LF_KFE
- removed link C_LH_FOOT
- removed link C_LH_HAA
- removed link C_LH_HFE
- removed link C_LH_KFE
- removed link C_RF_FOOT
- removed link C_RF_HAA
- removed link C_RF_HFE
- removed link C_RF_KFE
- removed link C_RH_FOOT
- removed link C_RH_HAA
- removed link C_RH_HFE
- removed link C_RH_KFE
- removed link base_link
- removed link imu_link
- added link LF_FOOT, mass 0.07000000; collision sphere radius=0.019; visual mesh filename=package://colt/meshes/C_LF_FOOT.STL
- added link LF_calf, mass 0.11881926; collision mesh filename=package://colt/meshes/C_LF_KFE.STL; visual mesh filename=package://colt/meshes/C_LF_KFE.STL
- added link LF_hip, mass 0.64335910; collision mesh filename=package://colt/meshes/C_LF_HAA.STL; visual mesh filename=package://colt/meshes/C_LF_HAA.STL
- added link LF_thigh, mass 0.79839719; collision mesh filename=package://colt/meshes/C_LF_HFE.STL; visual mesh filename=package://colt/meshes/C_LF_HFE.STL
- added link LH_FOOT, mass 0.07000000; collision sphere radius=0.019; visual mesh filename=package://colt/meshes/C_LH_FOOT.STL
- added link LH_calf, mass 0.11881926; collision mesh filename=package://colt/meshes/C_LH_KFE.STL; visual mesh filename=package://colt/meshes/C_LH_KFE.STL
- added link LH_hip, mass 0.64335910; collision mesh filename=package://colt/meshes/C_LH_HAA.STL; visual mesh filename=package://colt/meshes/C_LH_HAA.STL
- added link LH_thigh, mass 0.79839719; collision mesh filename=package://colt/meshes/C_LH_HFE.STL; visual mesh filename=package://colt/meshes/C_LH_HFE.STL
- added link RF_FOOT, mass 0.07000000; collision sphere radius=0.019; visual mesh filename=package://colt/meshes/C_RF_FOOT.STL
- added link RF_calf, mass 0.11881926; collision mesh filename=package://colt/meshes/C_RF_KFE.STL; visual mesh filename=package://colt/meshes/C_RF_KFE.STL
- added link RF_hip, mass 0.64335910; collision mesh filename=package://colt/meshes/C_RF_HAA.STL; visual mesh filename=package://colt/meshes/C_RF_HAA.STL
- added link RF_thigh, mass 0.79839719; collision mesh filename=package://colt/meshes/C_RF_HFE.STL; visual mesh filename=package://colt/meshes/C_RF_HFE.STL
- added link RH_FOOT, mass 0.07000000; collision sphere radius=0.019; visual mesh filename=package://colt/meshes/C_RH_FOOT.STL
- added link RH_calf, mass 0.11881926; collision mesh filename=package://colt/meshes/C_RH_KFE.STL; visual mesh filename=package://colt/meshes/C_RH_KFE.STL
- added link RH_hip, mass 0.64335910; collision mesh filename=package://colt/meshes/C_RH_HAA.STL; visual mesh filename=package://colt/meshes/C_RH_HAA.STL
- added link RH_thigh, mass 0.79839719; collision mesh filename=package://colt/meshes/C_RH_HFE.STL; visual mesh filename=package://colt/meshes/C_RH_HFE.STL
- added link base, mass 2.75268889; collision mesh filename=package://colt/meshes/base_link.STL; visual mesh filename=package://colt/meshes/base_link.STL
- added link base_imu, mass 0.00800000; collision mesh filename=package://colt/meshes/imu_link.STL; visual mesh filename=package://colt/meshes/imu_link.STL
Joints:
- removed joint IMU_fixed
- removed joint LF_FOOT_fixed
- removed joint LH_FOOT_fixed
- removed joint RF_FOOT_fixed
- removed joint RH_FOOT_fixed
- added joint LF_foot_fixed: type fixed, parent LF_calf, child LF_FOOT, origin xyz=0.17522 0 -0.22084 rpy=0 0 0
- added joint LH_foot_fixed: type fixed, parent LH_calf, child LH_FOOT, origin xyz=0.175215215481091 0 -0.220837258839277 rpy=0 0 0
- added joint RF_foot_fixed: type fixed, parent RF_calf, child RF_FOOT, origin xyz=0.17521 0 -0.22084 rpy=0 0 0
- added joint RH_foot_fixed: type fixed, parent RH_calf, child RH_FOOT, origin xyz=0.175213793021927 0 -0.220838115693587 rpy=0 0 0
- added joint base_imu_joint: type fixed, parent base, child base_imu, origin xyz=0 0 0.023 rpy=0 0 0
- joint LF_HAA: child C_LF_HAA -> LF_hip; parent base_link -> base
- joint LF_HFE: child C_LF_HFE -> LF_thigh; parent C_LF_HAA -> LF_hip
- joint LF_KFE: child C_LF_KFE -> LF_calf; parent C_LF_HFE -> LF_thigh
- joint LH_HAA: child C_LH_HAA -> LH_hip; parent base_link -> base
- joint LH_HFE: child C_LH_HFE -> LH_thigh; parent C_LH_HAA -> LH_hip
- joint LH_KFE: child C_LH_KFE -> LH_calf; parent C_LH_HFE -> LH_thigh
- joint RF_HAA: child C_RF_HAA -> RF_hip; parent base_link -> base
- joint RF_HFE: child C_RF_HFE -> RF_thigh; parent C_RF_HAA -> RF_hip
- joint RF_KFE: child C_RF_KFE -> RF_calf; parent C_RF_HFE -> RF_thigh
- joint RH_HAA: child C_RH_HAA -> RH_hip; parent base_link -> base
- joint RH_HFE: child C_RH_HFE -> RH_thigh; parent C_RH_HAA -> RH_hip
- joint RH_KFE: child C_RH_KFE -> RH_calf; parent C_RH_HFE -> RH_thigh

Commit message: urdf更新，关节角度转动方向与实机一致，并在rviz中验证

File: src/colt/urdf/colt.urdf (robot description, URDF)
Before this commit: robot colt, 18 links, 17 joints
Links:
- removed link base_link
- removed link imu_link
- added link baselink, mass 3.78620000; collision mesh filename=package://colt/meshes/baselink.STL; visual mesh filename=package://colt/meshes/baselink.STL
- added link imu_Link, mass 0.00800000; collision mesh filename=package://colt/meshes/imu_Link.STL; visual mesh filename=package://colt/meshes/imu_Link.STL
- link C_LF_FOOT: geometry collision mesh filename=package://colt/meshes/C_LF_FOOT.STL; visual mesh filename=package://colt/meshes/C_LF_FOOT.STL
- link C_LF_HAA: mass 0.64335910 -> 0.65477754
- link C_LF_HFE: mass 0.79839719 -> 0.80430000
- link C_LF_KFE: mass 0.11881926 -> 0.09520000
- link C_LH_FOOT: geometry collision mesh filename=package://colt/meshes/C_LH_FOOT.STL; visual mesh filename=package://colt/meshes/C_LH_FOOT.STL
- link C_LH_HAA: mass 0.64335910 -> 0.65477754
- link C_LH_HFE: mass 0.79839719 -> 0.80430000
- link C_LH_KFE: mass 0.11881926 -> 0.09520000
- link C_RF_FOOT: geometry collision mesh filename=package://colt/meshes/C_RF_FOOT.STL; visual mesh filename=package://colt/meshes/C_RF_FOOT.STL
- link C_RF_HAA: mass 0.64335910 -> 0.65477754
- link C_RF_HFE: mass 0.79839719 -> 0.80510000
- link C_RF_KFE: mass 0.11881926 -> 0.09520000
- link C_RH_FOOT: geometry collision mesh filename=package://colt/meshes/C_RH_FOOT.STL; visual mesh filename=package://colt/meshes/C_RH_FOOT.STL
- link C_RH_HAA: mass 0.64335910 -> 0.65477754
- link C_RH_HFE: mass 0.79839719 -> 0.80510000
- link C_RH_KFE: mass 0.11881926 -> 0.09520000
Joints:
- removed joint LF_FOOT_fixed
- removed joint LH_FOOT_fixed
- removed joint RF_FOOT_fixed
- removed joint RH_FOOT_fixed
- added joint LF_FOOT: type fixed, parent C_LF_KFE, child C_LF_FOOT, origin xyz=0.166232058395859 0 -0.166232410966886 rpy=0 0 0, axis 0 0 0
- added joint LH_FOOT: type fixed, parent C_LH_KFE, child C_LH_FOOT, origin xyz=0.166231482609425 0 -0.166232355223461 rpy=0 0 0, axis 0 0 0
- added joint RF_FOOT: type fixed, parent C_RF_KFE, child C_RF_FOOT, origin xyz=0.166232363094352 0 -0.16623147473847 rpy=0 0 0, axis 0 0 0
- added joint RH_FOOT: type fixed, parent C_RH_KFE, child C_RH_FOOT, origin xyz=0.166232363094353 0 -0.166231474738594 rpy=0 0 0, axis 0 0 0
- joint IMU_fixed: child imu_link -> imu_Link; origin xyz=0 0 0.023 rpy=0 0 0 -> xyz=0 0 0.0215 rpy=0 0 0; parent base_link -> baselink
- joint LF_HAA: axis -1 0 0 -> 1 0 0; limit lower=-6.28 upper=6.28 effort=100 velocity=100 -> lower=-3.14 upper=3.14 effort=50 velocity=50; origin xyz=0.1561 0.0699999999999992 0.0500000000000014 rpy=0 0 0 -> xyz=0.1311 0.06 0.0585 rpy=0 0 0; parent base_link -> baselink
- joint LF_HFE: axis 0 -1 0 -> 0 1 0; limit lower=-6.28 upper=6.28 effort=100 velocity=100 -> lower=-3.14 upper=3.14 effort=50 velocity=50; origin xyz=0.0555001125555474 0.0978000000000008 0 rpy=0 0 0 -> xyz=0.0555 0.0898 0 rpy=0 0 0
- joint LF_KFE: limit lower=-6.28 upper=6.28 effort=100 velocity=100 -> lower=-3.14 upper=3.14 effort=50 velocity=50; origin xyz=-0.25 0 0 rpy=0 0 0 -> xyz=-0.2 0 0 rpy=0 0 0
- joint LH_HAA: axis 1 0 0 -> -1 0 0; limit lower=-6.28 upper=6.28 effort=100 velocity=100 -> lower=-3.14 upper=3.14 effort=50 velocity=50; origin xyz=-0.1561 0.07 0.05 rpy=0 0 0 -> xyz=-0.1311 0.06 0.0585 rpy=0 0 0; parent base_link -> baselink
- joint LH_HFE: limit lower=-6.28 upper=6.28 effort=100 velocity=100 -> lower=-3.14 upper=3.14 effort=50 velocity=50; origin xyz=-0.0554998874444527 0.097799999999991 0 rpy=0 0 0 -> xyz=-0.0555000795883689 0.0898000000000003 0 rpy=0 0 0
- joint LH_KFE: limit lower=-6.28 upper=6.28 effort=100 velocity=100 -> lower=-3.14 upper=3.14 effort=50 velocity=50; origin xyz=-0.249999999999123 0 0 rpy=0 0 0 -> xyz=-0.2 0 0 rpy=0 0 0
- joint RF_HAA: axis -1 0 0 -> 1 0 0; limit lower=-6.28 upper=6.28 effort=100 velocity=100 -> lower=-3.14 upper=3.14 effort=50 velocity=50; origin xyz=0.156099999999998 -0.0700000000000004 0.0500000000000079 rpy=0 0 0 -> xyz=0.1311 -0.06 0.0585 rpy=0 0 0; parent base_link -> baselink
- joint RF_HFE: axis 0 1 0 -> 0 -1 0; limit lower=-6.28 upper=6.28 effort=100 velocity=100 -> lower=-3.14 upper=3.14 effort=50 velocity=50; origin xyz=0.0554998874444546 -0.0977999999999988 0 rpy=0 0 0 -> xyz=0.0555000795883688 -0.0897999999999995 0 rpy=0 0 0
- joint RF_KFE: axis 0 1 0 -> 0 -1 0; limit lower=-6.28 upper=6.28 effort=100 velocity=100 -> lower=-3.14 upper=3.14 effort=50 velocity=50; origin xyz=-0.249999999995038 0 0 rpy=0 0 0 -> xyz=-0.2 0 0 rpy=0 0 0
- joint RH_HAA: axis 1 0 0 -> -1 0 0; limit lower=-6.28 upper=6.28 effort=100 velocity=100 -> lower=-3.14 upper=3.14 effort=50 velocity=50; origin xyz=-0.1561 -0.07 0.05 rpy=0 0 0 -> xyz=-0.1311 -0.06 0.0585 rpy=0 0 0; parent base_link -> baselink
- joint RH_HFE: limit lower=-6.28 upper=6.28 effort=100 velocity=100 -> lower=-3.14 upper=3.14 effort=50 velocity=50; origin xyz=-0.055500112553648 -0.0978000000000028 0 rpy=0 0 0 -> xyz=-0.0555003046991673 -0.0898000000000001 0 rpy=0 0 0
- joint RH_KFE: axis 0 1 0 -> 0 -1 0; limit lower=-6.28 upper=6.28 effort=100 velocity=100 -> lower=-3.14 upper=3.14 effort=50 velocity=50; origin xyz=-0.250000000000101 0 0 rpy=0 0 0 -> xyz=-0.2 0 0 rpy=0 0 0

Commit message: urdf文件导出与宇树的碰撞模型对齐

File: src/colt/urdf/colt.urdf (robot description, URDF)
Before this commit: robot colt, 18 links, 17 joints
Links:
- link C_LF_FOOT: mass 0.07000000 -> 0.05000000; geometry collision sphere radius=0.019; visual mesh filename=package://colt/meshes/C_LF_FOOT.STL
- link C_LF_HAA: mass 0.65477754 -> 0.65469272; geometry collision cylinder length=0.09 radius=0.035; visual mesh filename=package://colt/meshes/C_LF_HAA.STL
- link C_LF_HFE: mass 0.80430000 -> 0.80510000; geometry collision box size=0.20 0.030 0.035; visual mesh filename=package://colt/meshes/C_LF_HFE.STL
- link C_LF_KFE: mass 0.09520000 -> 0.11520000; geometry collision box size=0.23 0.016 0.016; visual mesh filename=package://colt/meshes/C_LF_KFE.STL
- link C_LH_FOOT: mass 0.07000000 -> 0.05000000; geometry collision sphere radius=0.019; visual mesh filename=package://colt/meshes/C_LH_FOOT.STL
- link C_LH_HAA: mass 0.65477754 -> 0.65469272; geometry collision cylinder length=0.09 radius=0.035; visual mesh filename=package://colt/meshes/C_LH_HAA.STL
- link C_LH_HFE: mass 0.80430000 -> 0.80510000; geometry collision box size=0.20 0.030 0.035; visual mesh filename=package://colt/meshes/C_LH_HFE.STL
- link C_LH_KFE: mass 0.09520000 -> 0.11520000; geometry collision box size=0.23 0.016 0.016; visual mesh filename=package://colt/meshes/C_LH_KFE.STL
- link C_RF_FOOT: mass 0.07000000 -> 0.05000000; geometry collision sphere radius=0.019; visual mesh filename=package://colt/meshes/C_RF_FOOT.STL
- link C_RF_HAA: mass 0.65477754 -> 0.65469272; geometry collision cylinder length=0.09 radius=0.035; visual mesh filename=package://colt/meshes/C_RF_HAA.STL
- link C_RF_HFE: geometry collision box size=0.20 0.030 0.035; visual mesh filename=package://colt/meshes/C_RF_HFE.STL
- link C_RF_KFE: mass 0.09520000 -> 0.11520000; geometry collision box size=0.23 0.016 0.016; visual mesh filename=package://colt/meshes/C_RF_KFE.STL
- link C_RH_FOOT: mass 0.07000000 -> 0.05000000; geometry collision sphere radius=0.019; visual mesh filename=package://colt/meshes/C_RH_FOOT.STL
- link C_RH_HAA: mass 0.65477754 -> 0.65469272; geometry collision cylinder length=0.09 radius=0.035; visual mesh filename=package://colt/meshes/C_RH_HAA.STL
- link C_RH_HFE: geometry collision box size=0.20 0.030 0.035; visual mesh filename=package://colt/meshes/C_RH_HFE.STL
- link C_RH_KFE: mass 0.09520000 -> 0.11520000; geometry collision box size=0.23 0.016 0.016; visual mesh filename=package://colt/meshes/C_RH_KFE.STL
- link baselink: geometry collision box size=0.32 0.15 0.10; visual mesh filename=package://colt/meshes/baselink.STL
- link imu_Link: geometry collision box size=0.001 0.001 0.001; visual mesh filename=package://colt/meshes/imu_Link.STL
Joints:
- joint LF_FOOT: origin xyz=0.166232058395859 0 -0.166232410966886 rpy=0 0 0 -> xyz=0 0 -0.229999807853034 rpy=0 0 0
- joint LF_HAA: limit lower=-3.14 upper=3.14 effort=50 velocity=50 -> lower=-3.14 upper=3.14 effort=30 velocity=30
- joint LF_HFE: limit lower=-3.14 upper=3.14 effort=50 velocity=50 -> lower=-3.14 upper=3.14 effort=30 velocity=30
- joint LF_KFE: limit lower=-3.14 upper=3.14 effort=50 velocity=50 -> lower=-3.14 upper=3.14 effort=30 velocity=30; origin xyz=-0.2 0 0 rpy=0 0 0 -> xyz=0 0 -0.2 rpy=0 0 0
- joint LH_FOOT: origin xyz=0.166231482609425 0 -0.166232355223461 rpy=0 0 0 -> xyz=0 0 -0.229999999990562 rpy=0 0 0
- joint LH_HAA: axis -1 0 0 -> 1 0 0; limit lower=-3.14 upper=3.14 effort=50 velocity=50 -> lower=-3.14 upper=3.14 effort=30 velocity=30
- joint LH_HFE: limit lower=-3.14 upper=3.14 effort=50 velocity=50 -> lower=-3.14 upper=3.14 effort=30 velocity=30; origin xyz=-0.0555000795883689 0.0898000000000003 0 rpy=0 0 0 -> xyz=-0.0555 0.0898 0 rpy=0 0 0
- joint LH_KFE: limit lower=-3.14 upper=3.14 effort=50 velocity=50 -> lower=-3.14 upper=3.14 effort=30 velocity=30; origin xyz=-0.2 0 0 rpy=0 0 0 -> xyz=0 0 -0.2 rpy=0 0 0
- joint RF_FOOT: origin xyz=0.166232363094352 0 -0.16623147473847 rpy=0 0 0 -> xyz=0 0 -0.23 rpy=0 0 0
- joint RF_HAA: limit lower=-3.14 upper=3.14 effort=50 velocity=50 -> lower=-3.14 upper=3.14 effort=30 velocity=30
- joint RF_HFE: axis 0 -1 0 -> 0 1 0; limit lower=-3.14 upper=3.14 effort=50 velocity=50 -> lower=-3.14 upper=3.14 effort=30 velocity=30; origin xyz=0.0555000795883688 -0.0897999999999995 0 rpy=0 0 0 -> xyz=0.0555 -0.0898 0 rpy=0 0 0
- joint RF_KFE: axis 0 -1 0 -> 0 1 0; limit lower=-3.14 upper=3.14 effort=50 velocity=50 -> lower=-3.14 upper=3.14 effort=30 velocity=30; origin xyz=-0.2 0 0 rpy=0 0 0 -> xyz=0 0 -0.2 rpy=0 0 0
- joint RH_FOOT: origin xyz=0.166232363094353 0 -0.166231474738594 rpy=0 0 0 -> xyz=0 0 -0.23 rpy=0 0 0
- joint RH_HAA: axis -1 0 0 -> 1 0 0; limit lower=-3.14 upper=3.14 effort=50 velocity=50 -> lower=-3.14 upper=3.14 effort=30 velocity=30
- joint RH_HFE: axis 0 -1 0 -> 0 1 0; limit lower=-3.14 upper=3.14 effort=50 velocity=50 -> lower=-3.14 upper=3.14 effort=30 velocity=30; origin xyz=-0.0555003046991673 -0.0898000000000001 0 rpy=0 0 0 -> xyz=-0.0555 -0.0898 0 rpy=0 0 0
- joint RH_KFE: axis 0 -1 0 -> 0 1 0; limit lower=-3.14 upper=3.14 effort=50 velocity=50 -> lower=-3.14 upper=3.14 effort=30 velocity=30; origin xyz=-0.2 0 0 rpy=0 0 0 -> xyz=0 0 -0.2 rpy=0 0 0
